File: hardware/otto.sch (EAGLE design)
At the start: 71 parts, among them U1 BLU, U2 TPS61230DRCR, U3 PAM8302AASCR, U4 BMX160

Commit message: Hardware changes for v1B, see readme file
Parts:
- removed BUZZ: (no value), otto:PINHD-1X2
- removed D8: TPSQTP15R, otto:TPSQTP15R
- removed Q1: (no value), otto:MOSFET-NREFLOW
- added C25: 100u, otto:CAP_CERAMIC_1206
- added C26: 100n, otto:CAP_CERAMIC_0603
- added D2, D3: TPSQTP10R, otto:TPSQTP10R
- added D9: TPSQTP15R, otto:TPSQTP15R
- added U5: TPS2115AIPWRQ1-SON8, otto:TPS2115AIPWRQ1-SON8
- added U6: MIC-PDM-MP23DB01HPTR, otto:MIC-PDM-MP23DB01HPTR
- C11: value 100n -> 10u
- R6: value 100k -> 1k
Connections:
- removed net D24/MISO: D24.TP, U1.D24/MISO
- removed net D26/SCLK: D26.TP, U1.D26/SCLK
- removed net D4/BUZZ_CTRL: D4.TP, Q1.G, R6.1, U1.D4
- removed net D8/SM6: D8.TP, S6.3, U1.D9
- removed net N$19: BUZZ.2, Q1.D
- new net D24/MISO/MDAT: D24.TP, U1.D24/MISO, U6.DATA
- new net D26/SCLK/MCLK: D26.TP, U1.D26/SCLK, U6.CLOCK
- new net D4: D4.TP, U1.D4
- new net D9/SM6: D9.TP, S6.3, U1.D9
- new net N$6: D2.TP, U5.D0
- new net N$8: R6.2, U5.ILIM
- new net VIN: C1.1, C8.1, L1.1, U2.VIN, U5.OUT
- net 3V3: now also C26.1, U6.VDD
- net 5V0: now also C25.2; no longer BUZZ.1
- net GND: now also C25.1, C26.2, D3.TP, R6.1, U5.D1, U5.GND, U6.GND, U6.L/R; no longer Q1.S, R6.2
- net VBAT: now also U5.IN2; no longer C1.1, C8.1, L1.1, U2.VIN
- net VBUS: now also U5.IN1
Other:
- note added: "Microphone"
- note added: "Power Selector"
- note removed: "Buzzer"
- moved on the sheet: BATT, C9, LED, PWR-SW, R6, TC1, U1

Commit message: Lots of PCB changes v2 (see hardware readme)
Parts:
- removed D3: TPSQTP10R, otto:TPSQTP10R
- added 3V3, GND, PEN, RST, SCL, SDA, VBS, VBT: TPSQTP10R, otto:TPSQTP10R
- added C27, C28, C29: 100n, otto:CAP_CERAMIC_0603
- added C30, C31: 10u, otto:CAP_CERAMIC_0603
- added H1, H2: (no value), otto:VLP-XXX-X
- added PIR: (no value), otto:PINHD-1X3
- added R10: 4.7, otto:RESISTOR_0603
- added R8, R9: 100k, otto:RESISTOR_0603
- added U13: SHT4X, otto:SHT4X
- added U15: LPS22HB, otto:LPS22HB
- added U17: SGP41, otto:SGP41
- added U7: SPK0641HT4H, otto:SPK0641HT4H
- C18, C5: value 10u -> 100n
- D0, D1, D15, D16, D17, D18, D19, D24, D25, D26, D4, D5, D6, D7, D9: value TPSQTP15R -> TPSQTP10R; device otto:TPSQTP15R -> otto:TPSQTP10R
- D2: value TPSQTP10R -> SK6812MINI; device otto:TPSQTP10R -> otto:SK6812MINI
- U5: value TPS2115AIPWRQ1-SON8 -> TPS2115AIPWRQ1; device otto:TPS2115AIPWRQ1-SON8 -> otto:TPS2115AIPWRQ1
- U6: value MIC-PDM-MP23DB01HPTR -> APDS-9250; device otto:MIC-PDM-MP23DB01HPTR -> otto:APDS-9250
Connections:
- removed net D0/IMU_INT: D0.TP, U1.D0/TXD, U4.INT1
- removed net D1/SPKR: D1.TP, U1.D1/RXD, VR1.E
- removed net D15/SM3: D15.TP, S3.3, U1.D15/A1
- removed net D16/SM2: D16.TP, S2.3, U1.D16/A2
- removed net D17/SM1: D17.TP, S1.3, U1.D17/A3
- removed net D18/USRF_ECHO: D18.TP, U1.D18/A4, USRF.3
- removed net D19/USRF_TRIG: D19.TP, U1.D19/A5, USRF.4
- removed net D25/MOSI: D25.TP, U1.D25/MOSI
- removed net D4: D4.TP, U1.D4
- removed net D7/TOUCH_INT: D7.TP, TOUCH.5, U1.D7
- removed net D9/SM6: D9.TP, S6.3, U1.D9
- removed net N$6: D2.TP, U5.D0
- new net 3V3_A: C30.1, R10.2, U17.VDD
- new net D0/USRF_TRIG: D0.TP, U1.D0/TXD, USRF.4
- new net D1/USRF_ECHO: D1.TP, U1.D1/RXD, USRF.3
- new net D15/SM6: D15.TP, S6.3, U1.D15/A1
- new net D16/SM3: D16.TP, S3.3, U1.D16/A2
- new net D17/SM2: D17.TP, S2.3, U1.D17/A3
- new net D18/SM1: D18.TP, S1.3, U1.D18/A4
- new net D19/PIR: D19.TP, R9.1, U1.D19/A5
- new net D25/MOSI/PIX: D2.DI, D25.TP, U1.D25/MOSI
- new net D4/SPKR: D4.TP, U1.D4, VR1.E
- new net D7/IMU_INT: D7.TP, U1.D7, U4.INT1
- new net D9/TOUCH_INT: D9.TP, TOUCH.5, U1.D9
- new net N$5: PIR.3, R8.2, R9.2
- net !RST: now also RST.TP
- net 3V3: now also 3V3.TP, C18.2, C27.1, C28.1, C29.1, C31.1, C5.1, D2.VDD, PIR.2, R10.1, U13.VDD, U15.CS, U15.VDD, U15.VDD_IO, U17.VDDH, U7.VDD
- net 5V0: no longer C18.2, C5.2
- net D22/SDA: now also SDA.TP, U13.SDA, U15.SDA/SDIO, U17.SDA, U6.SDA
- net D23/SCL: now also SCL.TP, U13.SCL, U15.SCL/SPC, U17.SCL, U6.SCL
- net D24/MISO/MDAT: now also U7.DATA; no longer U6.DATA
- net D26/SCLK/MCLK: now also U7.CLOCK; no longer U6.CLOCK
- net GND: now also C27.2, C28.2, C29.2, C30.2, C31.2, C5.2, D2.VSS, GND.TP, PIR.1, R8.1, U13.VSS, U15.GND, U15.SDO/SA0, U17.R, U17.VSS, U7.GND, U7.L/R; no longer C5.1, D3.TP, U6.L/R
- net PWR_EN: now also PEN.TP
- net VBAT: now also VBT.TP
- net VBUS: now also VBS.TP
Other:
- note added: "Air Pressure Sensor"
- note added: "Light Sensor"
- note added: "Neopixel LED"
- note added: "PIR Sensor"
- note added: "Temp/Humidity Sensor"
- note added: "VOC/Gas Sensor"
- note removed: "Battery Jack"
- moved on the sheet: BATT, C10, C11, C18, C19, C20, C21, C23, C24, C25, C26, C5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
